Commit message: 修改urdf文件，模型大小缩放调整

File: llama_ws/src/llama_pkg/urdf/llama_bot.urdf (robot description, URDF)
Before this commit: robot llama_bot, 5 links, 4 joints
Links:
- link base_link: geometry collision mesh filename=package://llama_pkg/meshes/base_link.STL scale=0.001 0.001 0.001; visual mesh filename=package://llama_pkg/meshes/base_link.STL scale=0.001 0.001 0.001
